File: STM32_Bluepill.kicad_pcb (KiCad board)
At the start: 2 copper layers, 41 x 31 mm, 32 parts, among them J1 USB_B_Micro, J2 Conn_01x04_Male, J3 Conn_01x04_Male, J4 Conn_01x04_Male, U1 STM32F103C8T6, U2 AMS1117-3.3, Y1 16MHz

Commit message: Silkscreen: Add custom duck image and board details on back of board
Parts:
- added Ducky: LOGO, LOGO, F.Cu at (164.6, 98.2)
- added REF**: OSHW-Logo2_7.3x6mm_SilkScreen, Symbol:OSHW-Logo2_7.3x6mm_SilkScreen, B.Cu at (180.1, 83.8)
- added REF**: KiCad-Logo2_5mm_SilkScreen, Symbol:KiCad-Logo2_5mm_SilkScreen, B.Cu at (167.0, 99.6)
Other:
- board text added: "Designed by Michael Ly github.com/Michael-Q-Ly"
- board text added: "Rev. A Dec 17, 2022"
- board text added: "STM32 Blue Pill (Clone)"
- board text added: "STM32 Blue Pill Clone - UART - SWD - I2C - 64 KiB Flash - 20 KiB SRAM"
